File: sch/batteryCase.sch (EAGLE design)
At the start: 7 parts, among them X1 C-GRID-04-70553

Commit message: Fine tuning the 3LR12 board layout
Parts:
- JP1: value FIXED GND -> LED!
- JP2: value FIXED PWR -> RUN!
- S1: value RUN -> RUN/LED
Connections:
- net N$2: now also S12.S
- net N$3: now also S11.S
Other:
- moved on the sheet: S1
Changed lines of the file:
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@@
 <parts>
 <part name="F1" library="special" deviceset="FUSE" device="" value="1A"/>
-<part name="S1" library="switch" deviceset="M9040P2" device="" value="RUN"/>
+<part name="S1" library="switch" deviceset="M9040P2" device="" value="RUN/LED"/>
 <part name="PAD1" library="wirepad" deviceset="SMD5" device="" value="+4V5"/>
 <part name="PAD2" library="wirepad" deviceset="SMD5" device="" value="0V"/>
 <part name="X1" library="con-molex" deviceset="C-GRID-04" device="-70553"/>
-<part name="JP1" library="pinhead" deviceset="PINHD-1X2" device="/90" value="FIXED GND"/>
-<part name="JP2" library="pinhead" deviceset="PINHD-1X2" device="/90" value="FIXED PWR"/>
+<part name="JP1" library="pinhead" deviceset="PINHD-1X2" device="/90" value="LED!"/>
+<part name="JP2" library="pinhead" deviceset="PINHD-1X2" device="/90" value="RUN!"/>
 </parts>
 <sheets>
@@
 <instances>
 <instance part="F1" gate="G$1" x="30.48" y="60.96"/>
-<instance part="S1" gate="2" x="53.34" y="50.8" rot="R270"/>
-<instance part="S1" gate="1" x="53.34" y="63.5" rot="R270"/>
+<instance part="S1" gate="2" x="50.8" y="50.8" rot="R270"/>
+<instance part="S1" gate="1" x="50.8" y="63.5" rot="R270"/>
 <instance part="PAD1" gate="1" x="10.16" y="60.96"/>
 <instance part="PAD2" gate="1" x="10.16" y="50.8"/>
@@
 <junction x="66.04" y="45.72"/>
 <pinref part="S1" gate="2" pin="P"/>
-<wire x1="43.18" y1="50.8" x2="48.26" y2="50.8" width="0.1524" layer="91"/>
+<wire x1="43.18" y1="50.8" x2="45.72" y2="50.8" width="0.1524" layer="91"/>
 <junction x="43.18" y="50.8"/>
+<pinref part="S1" gate="2" pin="S"/>
+<wire x1="55.88" y1="48.26" x2="66.04" y2="48.26" width="0.1524" layer="91"/>
 </segment>
 </net>
@@
 <junction x="66.04" y="76.2"/>
 <junction x="66.04" y="73.66"/>
-<wire x1="43.18" y1="60.96" x2="48.26" y2="60.96" width="0.1524" layer="91"/>
+<wire x1="43.18" y1="60.96" x2="45.72" y2="60.96" width="0.1524" layer="91"/>
 <junction x="43.18" y="60.96"/>
 <pinref part="S1" gate="1" pin="P"/>
+<pinref part="S1" gate="1" pin="S"/>
+<wire x1="55.88" y1="58.42" x2="60.96" y2="58.42" width="0.1524" layer="91"/>
+<wire x1="60.96" y1="58.42" x2="60.96" y2="55.88" width="0.1524" layer="91"/>
+<wire x1="60.96" y1="55.88" x2="43.18" y2="55.88" width="0.1524" layer="91"/>
+<wire x1="43.18" y1="55.88" x2="43.18" y2="60.96" width="0.1524" layer="91"/>
 </segment>
 </net>
@@
 <wire x1="63.5" y1="60.96" x2="73.66" y2="60.96" width="0.1524" layer="91"/>
 <pinref part="S1" gate="1" pin="O"/>
-<wire x1="58.42" y1="63.5" x2="63.5" y2="63.5" width="0.1524" layer="91"/>
+<wire x1="55.88" y1="63.5" x2="63.5" y2="63.5" width="0.1524" layer="91"/>
 </segment>
 </net>
@@
 <wire x1="63.5" y1="58.42" x2="73.66" y2="58.42" width="0.1524" layer="91"/>
 <pinref part="S1" gate="2" pin="O"/>
-<wire x1="58.42" y1="53.34" x2="63.5" y2="53.34" width="0.1524" layer="91"/>
+<wire x1="55.88" y1="53.34" x2="63.5" y2="53.34" width="0.1524" layer="91"/>
 </segment>
 </net>

Commit message: Better fuse holder and clearances
Parts:
- F1: value 1A -> FUSEKS10H; device special:FUSE -> fuse:FUSEKS10H
Connections:
- net N$1: now also F1.2; no longer F1.1
- net N$3: now also F1.1; no longer F1.2
Changed lines of the file:
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@@
 <grid distance="0.1" unitdist="inch" unit="inch" style="lines" multiple="1" display="no" altdistance="0.01" altunitdist="inch" altunit="inch"/>
 <layers>
-<layer number="1" name="Top" color="4" fill="1" visible="no" active="no"/>
-<layer number="16" name="Bottom" color="1" fill="1" visible="no" active="no"/>
-<layer number="17" name="Pads" color="2" fill="1" visible="no" active="no"/>
-<layer number="18" name="Vias" color="2" fill="1" visible="no" active="no"/>
-<layer number="19" name="Unrouted" color="6" fill="1" visible="no" active="no"/>
-<layer number="20" name="Dimension" color="15" fill="1" visible="no" active="no"/>
-<layer number="21" name="tPlace" color="7" fill="1" visible="no" active="no"/>
-<layer number="22" name="bPlace" color="7" fill="1" visible="no" active="no"/>
-<layer number="23" name="tOrigins" color="15" fill="1" visible="no" active="no"/>
-<layer number="24" name="bOrigins" color="15" fill="1" visible="no" active="no"/>
-<layer number="25" name="tNames" color="7" fill="1" visible="no" active="no"/>
-<layer number="26" name="bNames" color="7" fill="1" visible="no" active="no"/>
-<layer number="27" name="tValues" color="7" fill="1" visible="no" active="no"/>
-<layer number="28" name="bValues" color="7" fill="1" visible="no" active="no"/>
+<layer number="1" name="Top" color="4" fill="1" visible="yes" active="no"/>
+<layer number="16" name="Bottom" color="1" fill="1" visible="yes" active="no"/>
+<layer number="17" name="Pads" color="2" fill="1" visible="yes" active="no"/>
+<layer number="18" name="Vias" color="2" fill="1" visible="yes" active="no"/>
+<layer number="19" name="Unrouted" color="6" fill="1" visible="yes" active="no"/>
+<layer number="20" name="Dimension" color="15" fill="1" visible="yes" active="no"/>
+<layer number="21" name="tPlace" color="7" fill="1" visible="yes" active="no"/>
+<layer number="22" name="bPlace" color="7" fill="1" visible="yes" active="no"/>
+<layer number="23" name="tOrigins" color="15" fill="1" visible="yes" active="no"/>
+<layer number="24" name="bOrigins" color="15" fill="1" visible="yes" active="no"/>
+<layer number="25" name="tNames" color="7" fill="1" visible="yes" active="no"/>
+<layer number="26" name="bNames" color="7" fill="1" visible="yes" active="no"/>
+<layer number="27" name="tValues" color="7" fill="1" visible="yes" active="no"/>
+<layer number="28" name="bValues" color="7" fill="1" visible="yes" active="no"/>
 <layer number="29" name="tStop" color="7" fill="3" visible="no" active="no"/>
 <layer number="30" name="bStop" color="7" fill="6" visible="no" active="no"/>
@@
 <layer number="35" name="tGlue" color="7" fill="4" visible="no" active="no"/>
 <layer number="36" name="bGlue" color="7" fill="5" visible="no" active="no"/>
-<layer number="37" name="tTest" color="7" fill="1" visible="no" active="no"/>
-<layer number="38" name="bTest" color="7" fill="1" visible="no" active="no"/>
+<layer number="37" name="tTest" color="7" fill="1" visible="yes" active="no"/>
+<layer number="38" name="bTest" color="7" fill="1" visible="yes" active="no"/>
 <layer number="39" name="tKeepout" color="4" fill="11" visible="no" active="no"/>
 <layer number="40" name="bKeepout" color="1" fill="11" visible="no" active="no"/>
@@
 <layer number="44" name="Drills" color="7" fill="1" visible="no" active="no"/>
 <layer number="45" name="Holes" color="7" fill="1" visible="no" active="no"/>
-<layer number="46" name="Milling" color="3" fill="1" visible="no" active="no"/>
-<layer number="47" name="Measures" color="7" fill="1" visible="no" active="no"/>
-<layer number="48" name="Document" color="7" fill="1" visible="no" active="no"/>
-<layer number="49" name="Reference" color="7" fill="1" visible="no" active="no"/>
-<layer number="51" name="tDocu" color="7" fill="1" visible="no" active="no"/>
-<layer number="52" name="bDocu" color="7" fill="1" visible="no" active="no"/>
+<layer number="46" name="Milling" color="3" fill="1" visible="yes" active="no"/>
+<layer number="47" name="Measures" color="7" fill="1" visible="yes" active="no"/>
+<layer number="48" name="Document" color="7" fill="1" visible="yes" active="no"/>
+<layer number="49" name="Reference" color="7" fill="1" visible="yes" active="no"/>
+<layer number="51" name="tDocu" color="7" fill="1" visible="yes" active="no"/>
+<layer number="52" name="bDocu" color="7" fill="1" visible="yes" active="no"/>
 <layer number="90" name="Modules" color="5" fill="1" visible="yes" active="yes"/>
 <layer number="91" name="Nets" color="2" fill="1" visible="yes" active="yes"/>
@@
 </classes>
 <parts>
-<part name="F1" library="special" deviceset="FUSE" device="" value="1A"/>
 <part name="S1" library="switch" deviceset="M9040P2" device="" value="RUN/LED"/>
 <part name="PAD1" library="wirepad" deviceset="SMD5" device="" value="+4V5"/>
@@
 <part name="JP1" library="pinhead" deviceset="PINHD-1X2" device="/90" value="LED!"/>
 <part name="JP2" library="pinhead" deviceset="PINHD-1X2" device="/90" value="RUN!"/>
+<part name="F1" library="fuse" deviceset="FUSE" device="KS10H"/>
 </parts>
 <sheets>
@@
 </plain>
 <instances>
-<instance part="F1" gate="G$1" x="30.48" y="60.96"/>
 <instance part="S1" gate="2" x="50.8" y="50.8" rot="R270"/>
 <instance part="S1" gate="1" x="50.8" y="63.5" rot="R270"/>
@@
 <instance part="JP1" gate="G$1" x="78.74" y="45.72"/>
 <instance part="JP2" gate="G$1" x="78.74" y="73.66"/>
+<instance part="F1" gate="G$1" x="30.48" y="60.96" rot="R180"/>
 </instances>
 <busses>
 </busses>
 <nets>
-<net name="N$1" class="0">
-<segment>
-<pinref part="PAD1" gate="1" pin="P"/>
-<pinref part="F1" gate="G$1" pin="1"/>
-<wire x1="12.7" y1="60.96" x2="22.86" y2="60.96" width="0.1524" layer="91"/>
-</segment>
-</net>
 <net name="N$2" class="0">
 <segment>
@@
 <net name="N$3" class="0">
 <segment>
-<pinref part="F1" gate="G$1" pin="2"/>
-<wire x1="35.56" y1="60.96" x2="43.18" y2="60.96" width="0.1524" layer="91"/>
 <pinref part="JP2" gate="G$1" pin="1"/>
 <wire x1="76.2" y1="76.2" x2="66.04" y2="76.2" width="0.1524" layer="91"/>
@@
 <wire x1="60.96" y1="55.88" x2="43.18" y2="55.88" width="0.1524" layer="91"/>
 <wire x1="43.18" y1="55.88" x2="43.18" y2="60.96" width="0.1524" layer="91"/>
+<pinref part="F1" gate="G$1" pin="1"/>
+<wire x1="35.56" y1="60.96" x2="43.18" y2="60.96" width="0.1524" layer="91"/>
 </segment>
 </net>
@@
 </segment>
 </net>
+<net name="N$1" class="0">
+<segment>
+<pinref part="PAD1" gate="1" pin="P"/>
+<pinref part="F1" gate="G$1" pin="2"/>
+<wire x1="12.7" y1="60.96" x2="25.4" y2="60.96" width="0.1524" layer="91"/>
+</segment>
+</net>
